Commit message: Adding a camera and somechanges to the lidar to make it more similar to my old package

File: urdf/two_wheeled_robot_nav2.urdf (robot description, URDF)
Before this commit: robot two_wheeled_robot, 5 links, 4 joints
Links:
- added link camera_link; collision box size=0.07 0.3 0.09; visual box size=0.07 0.3 0.09
Joints:
- added joint camera_joint: type fixed, parent base_link, child camera_link, origin xyz=${base_length/2} 0 ${base_height/7} rpy=0 0 0

Commit message: moved Wheels to the front, deleted IMU to make simulation faster, deleted meshes to make simulation faster

File: urdf/two_wheeled_robot_nav2.urdf (robot description, URDF)
Before this commit: robot two_wheeled_robot, 6 links, 5 joints
Links:
- removed link imu_link
- link base_link: geometry collision box size=${base_length} ${base_width} ${base_height}; visual box size=${base_length} ${base_width} ${base_height}
- link lidar_link: mass 0.125 -> None; geometry collision cylinder length=${lidar_height} radius=${lidar_radius}; visual cylinder length=${lidar_height} radius=${lidar_radius}
Joints:
- removed joint imu_joint
- joint caster_joint: origin xyz=${caster_xoff} 0.0 ${-(base_height/2)} rpy=0 0 0 -> xyz=${-(caster_xoff)} 0.0 ${-(base_height/2)} rpy=0 0 0
- joint lidar_joint: origin xyz=0.215 0.0 0.30 rpy=0 0 0 -> xyz=0.0 0.0 ${base_height} rpy=0 0 0

Commit message: Going back to a previous version of the robot with the wheels to the front, because previous changes produced an error where there robot could not move correctly. The IMU was deleted. Now the robot moves correctly, it has a camera and a very long lidar.

File: urdf/two_wheeled_robot_nav2.urdf (robot description, URDF)
Before this commit: robot two_wheeled_robot, 5 links, 4 joints
Links:
- link base_link: geometry collision box size=${base_length} ${base_width} ${base_height}; visual mesh filename=file://$(find two_wheeled_robot)/meshes/robot_base.stl
- link lidar_link: mass None -> 0.125; geometry collision cylinder length=0.75 radius=0.0508; visual cylinder length=0.75 radius=0.0508
Joints:
- joint caster_joint: origin xyz=${-(caster_xoff)} 0.0 ${-(base_height/2)} rpy=0 0 0 -> xyz=${caster_xoff} 0.0 ${-(base_height/2)} rpy=0 0 0
- joint lidar_joint: origin xyz=0.0 0.0 ${base_height} rpy=0 0 0 -> xyz=0.215 0.0 0.30 rpy=0 0 0
